Commit message: 0430

File: urdf/humanoid.urdf (robot description, URDF)
Before this commit: robot humanoid, 13 links, 12 joints
Links:
- link Elbow_XL430_1: geometry collision mesh filename=package://avatar/meshes/Elbow_XL430_1.stl scale=0.001 0.001 0.001; visual mesh filename=package://avatar/meshes/Elbow_XL430_1.stl scale=0.001 0.001 0.001
- link Shoulder_Pitch_XM430_1: geometry collision mesh filename=package://avatar/meshes/Shoulder_Pitch_XM430_1.stl scale=0.001 0.001 0.001; visual mesh filename=package://avatar/meshes/Shoulder_Pitch_XM430_1.stl scale=0.001 0.001 0.001
- link Shoulder_Roll_XL430_1: geometry collision mesh filename=package://avatar/meshes/Shoulder_Roll_XL430_1.stl scale=0.001 0.001 0.001; visual mesh filename=package://avatar/meshes/Shoulder_Roll_XL430_1.stl scale=0.001 0.001 0.001
- link Shoulder_Yaw_XL430_1: geometry collision mesh filename=package://avatar/meshes/Shoulder_Yaw_XL430_1.stl scale=0.001 0.001 0.001; visual mesh filename=package://avatar/meshes/Shoulder_Yaw_XL430_1.stl scale=0.001 0.001 0.001
- link Wrist_Pitch_XL430_1: geometry collision mesh filename=package://avatar/meshes/Wrist_Pitch_XL430_1.stl scale=0.001 0.001 0.001; visual mesh filename=package://avatar/meshes/Wrist_Pitch_XL430_1.stl scale=0.001 0.001 0.001
- link Wrist_Yaw_XL430_1: geometry collision mesh filename=package://avatar/meshes/Wrist_Yaw_XL430_1.stl scale=0.001 0.001 0.001; visual mesh filename=package://avatar/meshes/Wrist_Yaw_XL430_1.stl scale=0.001 0.001 0.001
- link base_link: geometry collision mesh filename=package://avatar/meshes/base_link.stl scale=0.001 0.001 0.001; visual mesh filename=package://avatar/meshes/base_link.stl scale=0.001 0.001 0.001
- link fr12-h104_v1_1: geometry collision mesh filename=package://avatar/meshes/fr12-h104_v1_1.stl scale=0.001 0.001 0.001; visual mesh filename=package://avatar/meshes/fr12-h104_v1_1.stl scale=0.001 0.001 0.001
- link fr12-h104_v1_2_1: geometry collision mesh filename=package://avatar/meshes/fr12-h104_v1_2_1.stl scale=0.001 0.001 0.001; visual mesh filename=package://avatar/meshes/fr12-h104_v1_2_1.stl scale=0.001 0.001 0.001
- link fr12_h101_k_v1_1: geometry collision mesh filename=package://avatar/meshes/fr12_h101_k_v1_1.stl scale=0.001 0.001 0.001; visual mesh filename=package://avatar/meshes/fr12_h101_k_v1_1.stl scale=0.001 0.001 0.001
- link fr12_s102_k_v1_1: geometry collision mesh filename=package://avatar/meshes/fr12_s102_k_v1_1.stl scale=0.001 0.001 0.001; visual mesh filename=package://avatar/meshes/fr12_s102_k_v1_1.stl scale=0.001 0.001 0.001
- link humanoid_robot_arm_v2_lower_arm_conn_1_v2_1: geometry collision mesh filename=package://avatar/meshes/humanoid_robot_arm_v2_lower_arm_con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 scale=0.001 0.001 0.001; visual mesh filename=package://avatar/meshes/humanoid_robot_arm_v2_lower_arm_con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 scale=0.001 0.001 0.001
- link humanoid_robot_arm_v2_lower_arm_conn_2_v2_1: geometry collision mesh filename=package://avatar/meshes/humanoid_robot_arm_v2_lower_arm_con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 scale=0.001 0.001 0.001; visual mesh filename=package://avatar/meshes/humanoid_robot_arm_v2_lower_arm_con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 scale=0.001 0.001 0.001
